File: Untitled.kicad_sch (KiCad schematic)
At the start: 0 parts

Commit message: Schematic done
Parts:
- added C1: 1 uF, Capacitor_THT:CP_Radial_D5.0mm_P2.00mm, symbol Device:C_Polarized
- added C2: 0.01 uF, Capacitor_THT:C_Disc_D7.5mm_W2.5mm_P5.00mm, symbol Device:C
- added D1, D10, D2, D3, D4, D5, D6, D7, D8, D9: LED, LED_THT:LED_D3.0mm, symbol Device:LED
- added J1: Conn_01x02_Socket, Connector_PinHeader_2.54mm:PinHeader_1x02_P2.54mm_Vertical, symbol Connector:Conn_01x02_Socket
- added R1: 1k, Resistor_THT:R_Axial_DIN0207_L6.3mm_D2.5mm_P7.62mm_Horizontal, symbol Device:R
- added R2: 470, Resistor_THT:R_Axial_DIN0207_L6.3mm_D2.5mm_P7.62mm_Horizontal, symbol Device:R
- added RV1: 50k, Potentiometer_THT:Potentiometer_Vishay_T93YA_Vertical, symbol Device:R_Potentiometer
- added U1: NE555P, Package_DIP:DIP-8_W7.62mm, symbol Timer:NE555P
- added U2: 4017, imported:CD4017BE, symbol 4xxx:4017
Connections:
- new net: D1.1 (K), D10.1 (K), D2.1 (K), D3.1 (K), D4.1 (K), D5.1 (K), D6.1 (K), D7.1 (K), D8.1 (K), D9.1 (K), R2.1
- new net: D1.2 (A), U2.1 (Q5)
- new net: D2.2 (A), U2.10 (Q4)
- new net: D10.2 (A), U2.11 (Q9)
- new net: D5.2 (A), U2.2 (Q1)
- new net: D6.2 (A), U2.3 (Q0)
- new net: D4.2 (A), U2.4 (Q2)
- new net: D8.2 (A), U2.5 (Q6)
- new net: D7.2 (A), U2.6 (Q7)
- new net: D3.2 (A), U2.7 (Q3)
- new net: D9.2 (A), U2.9 (Q8)
- new net: R1.2, RV1.1, RV1.2, U1.7 (DISCH)
- new net: C2.1, U1.5 (CONT)
- new net +5V: J1.1 (Pin_1), R1.1, U1.4 (~{RST}), U1.8 (VCC), U2.16 (VDD)
- new net GND: C1.2, C2.2, J1.2 (Pin_2), R2.2, U1.1 (GND), U2.13 (CKEN), U2.15 (Reset), U2.8 (VSS)
- new net OUT: U1.3 (OUT)
- new net TR: C1.1, RV1.3, U1.2 (TRIG), U1.6 (THRES)
- no-connect marks 0 -> 1
